Commit message: Set the mesh scale and origin
Signed-off-by: Abdelhak Bougouffa <a.bougouffa@ez-wheel.com>

File: urdf/swd_starter_kit.urdf (robot description, URDF)
Before this commit: robot swd_starter_kit, 4 links, 3 joints
Links:
- link base_link: geometry collision mesh filename=package://swd_starter_kit_description/meshes/starter_kit.stl scale=0.001 0.001 0.001; visual mesh filename=package://swd_starter_kit_description/meshes/starter_kit.stl scale=0.001 0.001 0.001

Commit message: update to ROS2

File: urdf/swd_starter_kit.urdf (robot description, URDF)
Before this commit: robot swd_starter_kit, 7 links, 6 joints
Links:
- removed link lidar_link
- added link laser, mass 0.1; collision cylinder length=0.02 radius=0.035
Joints:
- removed joint base_lidar_link
- added joint base_laser: type fixed, parent base_link, child laser, origin xyz=0.05 0 0.2 rpy=0 0 0, axis 0 0 0
